Commit message: Update cubo.xacro

File: cubo_description/urdf/cubo.xacro (robot description, xacro)
@@ -13,5 +13,5 @@
     <origin xyz="0 0 0" rpy="0 0 0"/>
     <geometry>
-      <mesh filename="package://cubo_description/meshes/base_link.stl" scale="0.001 0.001 0.001"/>
+      <mesh filename="package://cubo_description/meshes/base_link.stl"/>
     </geometry>
     <material name="silver"/>
@@ -20,5 +20,5 @@
     <origin xyz="0 0 0" rpy="0 0 0"/>
     <geometry>
-      <mesh filename="package://cubo_description/meshes/base_link.stl" scale="0.001 0.001 0.001"/>
+      <mesh filename="package://cubo_description/meshes/base_link.stl"/>
     </geometry>
   </collision>
@@ -33,5 +33,5 @@
     <origin xyz="-0.0 -0.0 -2.3" rpy="0 0 0"/>
     <geometry>
-      <mesh filename="package://cubo_description/meshes/sail_link_1.stl" scale="0.001 0.001 0.001"/>
+      <mesh filename="package://cubo_description/meshes/sail_link_1.stl"/>
     </geometry>
     <material name="silver"/>
@@ -40,5 +40,5 @@
     <origin xyz="-0.0 -0.0 -2.3" rpy="0 0 0"/>
     <geometry>
-      <mesh filename="package://cubo_description/meshes/sail_link_1.stl" scale="0.001 0.001 0.001"/>
+      <mesh filename="package://cubo_description/meshes/sail_link_1.stl"/>
     </geometry>
   </collision>
@@ -53,5 +53,5 @@
     <origin xyz="-0.0 -0.0 -1.0" rpy="0 0 0"/>
     <geometry>
-      <mesh filename="package://cubo_description/meshes/mast_link_1.stl" scale="0.001 0.001 0.001"/>
+      <mesh filename="package://cubo_description/meshes/mast_link_1.stl"/>
     </geometry>
     <material name="silver"/>
@@ -60,9 +60,9 @@
     <origin xyz="-0.0 -0.0 -1.0" rpy="0 0 0"/>
     <geometry>
-      <mesh filename="package://cubo_description/meshes/mast_link_1.stl" scale="0.001 0.001 0.001"/>
+      <mesh filename="package://cubo_description/meshes/mast_link_1.stl"/>
     </geometry>
   </collision>
 </link>
-<joint name="joint2" type="continuous">
+<joint name="joint2" type="continous">
   <origin xyz="0.0 0.0 1.3" rpy="0 0 0"/>
   <parent link="mast_link_1"/>
