Commit message: Update stintboat.urdf
Added camera sensor on top of the mast.

File: stintboat_description/urdf/stintboat.urdf (robot description, URDF)
Before this commit: robot stintboat, 6 links, 5 joints
Links:
- added link camera_link, mass 1e-5; collision box size=0.05 0.05 0.05; visual box size=0.05 0.05 0.05
- link pole_link: mass 0.2 -> 0.042
- link rudder_link: mass 0.2 -> 0.691
Joints:
- added joint camera_joint: type fixed, parent mast_link, child camera_link, origin xyz=0.999 0 1.82 rpy=0 0 0, axis 0.0 1.0 0.0

Commit message: Update stintboat.urdf
Added IMU sensor.

File: stintboat_description/urdf/stintboat.urdf (robot description, URDF)
Before this commit: robot stintboat, 7 links, 6 joints
Links:
- added link imu_link, mass 1e-5; collision box size=0.05 0.05 0.05; visual box size=0.05 0.05 0.05
Joints:
- added joint imu_joint: type fixed, parent base_link, child imu_link, origin xyz=0.800 0.0 0.5, axis 1.0 0.0 0.0
- joint camera_joint: origin xyz=0.999 0 1.82 rpy=0 0 0 -> xyz=0.999 0.0 1.82

Commit message: Update stintboat.urdf

File: stintboat_description/urdf/stintboat.urdf (robot description, URDF)
Before this commit: robot stintboat, 8 links, 7 joints
Joints:
- joint base_mast_joint: limit lower=0.0 upper=0.0 effort=0.0 velocity=0.0 -> lower=-3.14 upper=3.14 effort=1000.0 velocity=0.5; origin xyz=0.00957 0 0.003 -> xyz=0.957 0.0 0.5 rpy=0 0 0
- joint base_pole_joint: axis 0.0 0.0 1.0 -> 0.0 0.0 1.8
- joint camera_joint: origin xyz=0.999 0.0 1.82 -> xyz=0.0 0.0 1.3
- joint mast_sail_joint: origin xyz=0.0 0.0 0.0080 -> xyz=0.0 0.0 1.3 rpy=0 0 0

Commit message: Update stintboat.urdf

File: stintboat_description/urdf/stintboat.urdf (robot description, URDF)
Before this commit: robot stintboat, 8 links, 7 joints
Links:
- link mast_link: mass 1.2864 -> 2.481072798172541
- link pole_link: mass 0.042 -> 0.23856469213197484
- link rudder_link: mass 0.691 -> 1.3349130842340802
Joints:
- joint base_pole_joint: axis 0.0 0.0 1.8 -> 0.0 0.0 -1.0; limit lower=0.0 upper=0.0 effort=0.0 velocity=0.0 -> lower=-3.14 upper=3.14 effort=1000.0 velocity=0.5; origin xyz=0.00175 0 0.0050 -> xyz=0.25 0.0 0.5 rpy=0.0 0.0 0.0
- joint pole_rudder_joint: axis 0.0 0.0 1.0 -> (none); origin xyz=0.00175 0 0.0050 -> xyz=0.0 0.0 -0.5 rpy=0.0 0.0 0.0

Commit message: Update stintboat.urdf

File: stintboat_description/urdf/stintboat.urdf (robot description, URDF)
Before this commit: robot stintboat, 8 links, 7 joints
Joints:
- joint base_mast_joint: limit lower=-3.14 upper=3.14 effort=1000.0 velocity=0.5 -> (none); type revolute -> continuous
- joint base_pole_joint: limit lower=-3.14 upper=3.14 effort=1000.0 velocity=0.5 -> (none); type revolute -> continuous

Commit message: Update stintboat.urdf

File: stintboat_description/urdf/stintboat.urdf (robot description, URDF)
Before this commit: robot stintboat, 8 links, 7 joints
Links:
- link sail_link: mass 24.592097 -> 17.799

Commit message: Update stintboat.urdf

File: stintboat_description/urdf/stintboat.urdf (robot description, URDF)
Before this commit: robot stintboat, 8 links, 7 joints
Links:
- link rudder_link: mass 1.3349130842340802 -> 0.481

Commit message: Update stintboat.urdf

File: stintboat_description/urdf/stintboat.urdf (robot description, URDF)
Before this commit: robot stintboat, 8 links, 7 joints
Links:
- link base_link: mass 204.1612 -> 204.15012580813698; geometry collision mesh filename=package://stintboat_description/meshes/hull.stl; visual mesh filename=package://stintboat_description/meshes/hull.stl
- link mast_link: geometry collision mesh filename=package://stintboat_description/meshes/mast.stl; visual mesh filename=package://stintboat_description/meshes/mast.stl
- link pole_link: mass 0.23856469213197484 -> 0.10602875205865538; geometry collision mesh filename=package://stintboat_description/meshes/pole.stl; visual mesh filename=package://stintboat_description/meshes/pole.stl
- link rudder_link: mass 0.481 -> 0.47077962067253687; geometry collision mesh filename=package://stintboat_description/meshes/rudder.stl; visual mesh filename=package://stintboat_description/meshes/rudder.stl
- link sail_link: mass 17.799 -> 17.798853424590863; geometry collision mesh filename=package://stintboat_description/meshes/sail.stl; visual mesh filename=package://stintboat_description/meshes/sail.stl
Joints:
- joint pole_rudder_joint: origin xyz=0.0 0.0 -0.5 rpy=0.0 0.0 0.0 -> xyz=0.0 0.0 -1.0 rpy=0.0 0.0 0.0
